Commit message: description:   refactoring of robot descriptions   add default teleop configurations

File: campero_description/urdf/campero.xacro (robot description, xacro)
@@ -5,5 +5,5 @@
    <xacro:macro name="campero" params="model mode prefix">
       <xacro:property name="conf" value="$(find campero_description)/config/campero_${model}.yaml" />
-      <xacro:property name="props" value="${load_yaml(conf)['/**']['ros__parameters']['base_info']}" />
+      <xacro:property name="props" value="${load_yaml(conf)}" />
       <!-- Link names -->
       <xacro:property name="base_link" value="${props['links']['base_link_name']}" />

Commit message: refactoring + add CI

File: campero_description/urdf/campero.xacro (robot description, xacro)
@@ -56,6 +56,12 @@
       <xacro:property name="rear_wheel_mass" value="6.5" />
       <xacro:property name="chassis_height" value="${min(front_wheel_radius,rear_wheel_radius)}" />
-      <xacro:property name="simulation_hardware_plugin" value="romea_mobile_base_gazebo/GazeboSystemInterface4WD"/>
-      <xacro:property name="live_hardware_plugin" value="alpo_hardware/AlpoHardware"/>
+      <xacro:if value="${model == 'rubber'}">
+         <xacro:property name="simulation_hardware_plugin" value="romea_mobile_base_gazebo/GazeboSystemInterface4WD"/>
+         <xacro:property name="live_hardware_plugin" value="campero_hardware/CamperoHardware4WD"/>
+      </xacro:if>
+      <xacro:if value="${model == 'mecanum'}">
+         <xacro:property name="simulation_hardware_plugin" value="romea_mobile_base_gazebo/GazeboSystemInterface4WMD"/>
+         <xacro:property name="live_hardware_plugin" value="campero_hardware/CamperoHardware4WMD"/>
+      </xacro:if>
       <xacro:chassis>
         <visual>

Commit message: split ros2_control from urdf remove robot state publisher

File: campero_description/urdf/campero.xacro (robot description, xacro)
@@ -1,6 +1,5 @@
 <?xml version="1.0"?>
 <robot name="campero" xmlns:xacro="http://www.ros.org/wiki/xacro">
-   <xacro:include filename="$(find romea_mobile_base_description)/urdf/base4WD.chassis.xacro"/>
-   <xacro:include filename="$(find romea_mobile_base_description)/ros2_control/base4WD.ros2_control.xacro"/>
+   <xacro:include filename="$(find romea_mobile_base_description)/urdf/base4WD.chassis.xacro" />
    <xacro:macro name="campero" params="model mode prefix">
       <xacro:property name="conf" value="$(find campero_description)/config/campero_${model}.yaml" />
@@ -8,19 +7,28 @@
       <!-- Link names -->
       <xacro:property name="base_link" value="${props['links']['base_link_name']}" />
-      <xacro:property name="base_footprint_link" value="${props['links']['base_footprint_link_name']}" />
+      <xacro:property name="base_footprint_link"
+         value="${props['links']['base_footprint_link_name']}" />
       <xacro:property name="inertial_link" value="${props['links']['inertial_link_name']}" />
-      <xacro:property name="front_left_wheel_spinning_link" value="${props['links']['front_left_wheel_spinning_link_name']}" />
-      <xacro:property name="front_right_wheel_spinning_link" value="${props['links']['front_right_wheel_spinning_link_name']}" />
-      <xacro:property name="rear_left_wheel_spinning_link" value="${props['links']['rear_left_wheel_spinning_link_name']}" />
-      <xacro:property name="rear_right_wheel_spinning_link" value="${props['links']['rear_right_wheel_spinning_link_name']}" />
+      <xacro:property name="front_left_wheel_spinning_link"
+         value="${props['links']['front_left_wheel_spinning_link_name']}" />
+      <xacro:property name="front_right_wheel_spinning_link"
+         value="${props['links']['front_right_wheel_spinning_link_name']}" />
+      <xacro:property name="rear_left_wheel_spinning_link"
+         value="${props['links']['rear_left_wheel_spinning_link_name']}" />
+      <xacro:property name="rear_right_wheel_spinning_link"
+         value="${props['links']['rear_right_wheel_spinning_link_name']}" />
       <!-- Joint names -->
-      <xacro:property name="base_footprint_joint" value="${props['joints']['base_footprint_joint_name']}" />
-      <xacro:property name="inertial_joint" value="${props['joints']['inertial_joint_name']}" />
-      <xacro:property name="front_left_wheel_steering_joint" value="${props['joints']['front_left_wheel_steering_joint_name']}" />
-      <xacro:property name="front_right_wheel_steering_joint" value="${props['joints']['front_right_wheel_steering_joint_name']}" />
-      <xacro:property name="front_left_wheel_spinning_joint" value="${props['joints']['front_left_wheel_spinning_joint_name']}" />
-      <xacro:property name="front_right_wheel_spinning_joint" value="${props['joints']['front_right_wheel_spinning_joint_name']}" />
-      <xacro:property name="rear_left_wheel_spinning_joint" value="${props['joints']['rear_left_wheel_spinning_joint_name']}" />
-      <xacro:property name="rear_right_wheel_spinning_joint" value="${props['joints']['rear_right_wheel_spinning_joint_name']}" />
+      <xacro:property name="base_footprint_joint"
+         value="${props['joints']['base_footprint_joint_name']}" />
+      <xacro:property name="inertial_joint"
+         value="${props['joints']['inertial_joint_name']}" />
+      <xacro:property name="front_left_wheel_spinning_joint"
+         value="${props['joints']['front_left_wheel_spinning_joint_name']}" />
+      <xacro:property name="front_right_wheel_spinning_joint"
+         value="${props['joints']['front_right_wheel_spinning_joint_name']}" />
+      <xacro:property name="rear_left_wheel_spinning_joint"
+         value="${props['joints']['rear_left_wheel_spinning_joint_name']}" />
+      <xacro:property name="rear_right_wheel_spinning_joint"
+         value="${props['joints']['rear_right_wheel_spinning_joint_name']}" />
       <!-- Base Properties -->
       <xacro:property name="aabb_length" value="${props['geometry']['aabb']['length']}" />
@@ -30,9 +38,13 @@
       <xacro:property name="aabb_center_y" value="${props['geometry']['aabb']['center'][1]}" />
       <xacro:property name="aabb_center_z" value="${props['geometry']['aabb']['center'][2]}" />
-      <xacro:property name="wheelbase" value="${props['geometry']['axles_distance']}"/>
-      <xacro:property name="front_track" value="${props['geometry']['front_axle']['wheels_distance']}"/>
-      <xacro:property name="rear_track" value="${props['geometry']['rear_axle']['wheels_distance']}"/>
-      <xacro:property name="track" value="${front_track}"/>
-      <xacro:property name="ground_clearance" value="${chassis_props['ground_clearance']}"/>
+      <xacro:property name="wheelbase"
+         value="${props['geometry']['axles_distance']}" />
+      <xacro:property name="front_track"
+         value="${props['geometry']['front_axle']['wheels_distance']}" />
+      <xacro:property name="rear_track"
+         value="${props['geometry']['rear_axle']['wheels_distance']}" />
+      <xacro:property name="track"
+         value="${front_track}" />
+      <xacro:property name="ground_clearance" value="${chassis_props['ground_clearance']}" />
       <xacro:property name="mass_body" value="${props['inertia']['mass']}" />
       <xacro:property name="mass_base" value="${props['inertia']['mass']}" />
@@ -40,45 +52,42 @@
       <xacro:property name="mass_center_y" value="${props['inertia']['center'][1]}" />
       <xacro:property name="mass_center_z" value="${props['inertia']['center'][2]}" />
-      <xacro:property name="ground_clearance" value="${props['geometry']['ground_clearance']}"/>
+      <xacro:property name="ground_clearance" value="${props['geometry']['ground_clearance']}" />
       <xacro:property name="body_reference_x" value="${props['control_point'][0]}" />
       <!-- Wheel Properties -->
-      <xacro:property name="front_hub_carrier_offset" value="${props['geometry']['front_axle']['wheels']['hub_carrier_offset']}" />
-      <xacro:property name="rear_hub_carrier_offset" value="${props['geometry']['rear_axle']['wheels']['hub_carrier_offset']}" />
-      <xacro:property name="front_wheel_radius" value="${props['geometry']['front_axle']['wheels']['radius']}" />
-      <xacro:property name="rear_wheel_radius" value="${props['geometry']['rear_axle']['wheels']['radius']}" />
-      <xacro:property name="front_wheel_width" value="${props['geometry']['front_axle']['wheels']['width']}" />
-      <xacro:property name="rear_wheel_width" value="${props['geometry']['rear_axle']['wheels']['width']}" />
+      <xacro:property name="front_hub_carrier_offset"
+         value="${props['geometry']['front_axle']['wheels']['hub_carrier_offset']}" />
+      <xacro:property name="rear_hub_carrier_offset"
+         value="${props['geometry']['rear_axle']['wheels']['hub_carrier_offset']}" />
+      <xacro:property name="front_wheel_radius"
+         value="${props['geometry']['front_axle']['wheels']['radius']}" />
+      <xacro:property name="rear_wheel_radius"
+         value="${props['geometry']['rear_axle']['wheels']['radius']}" />
+      <xacro:property name="front_wheel_width"
+         value="${props['geometry']['front_axle']['wheels']['width']}" />
+      <xacro:property name="rear_wheel_width"
+         value="${props['geometry']['rear_axle']['wheels']['width']}" />
       <xacro:property name="wheel_radius" value="${front_wheel_radius}" />
       <xacro:property name="wheel_width" value="${front_wheel_width}" />
-      <xacro:property name="maximal_wheel_speed" value="${props['wheels_speed_control']['command']['maximal_speed']}"/>
+      <xacro:property name="maximal_wheel_speed"
+         value="${props['wheels_speed_control']['command']['maximal_speed']}" />
       <xacro:property name="wheel_mass" value="6.5" />
       <xacro:property name="front_wheel_mass" value="6.5" />
       <xacro:property name="rear_wheel_mass" value="6.5" />
       <xacro:property name="chassis_height" value="${min(front_wheel_radius,rear_wheel_radius)}" />
-      <xacro:if value="${model == 'rubber'}">
-         <xacro:property name="simulation_hardware_plugin" value="romea_mobile_base_gazebo/GazeboSystemInterface4WD"/>
-         <xacro:property name="live_hardware_plugin" value="campero_hardware/CamperoHardware4WD"/>
-      </xacro:if>
-      <xacro:if value="${model == 'mecanum'}">
-         <xacro:property name="simulation_hardware_plugin" value="romea_mobile_base_gazebo/GazeboSystemInterface4WMD"/>
-         <xacro:property name="live_hardware_plugin" value="campero_hardware/CamperoHardware4WMD"/>
-      </xacro:if>
       <xacro:chassis>
-        <visual>
-<!--            <origin xyz="${aabb_center_x-body_reference_x} ${aabb_center_y}  ${aabb_center_z-chassis_height}" rpy="0 0 0" />-->
+         <visual>
+            <!--            <origin xyz="${aabb_center_x-body_reference_x} ${aabb_center_y}
+            ${aabb_center_z-chassis_height}" rpy="0 0 0" />-->
             <geometry>
-              <mesh filename="package://campero_description/meshes/chassis.stl"/>
+               <mesh filename="package://campero_description/meshes/chassis.stl" />
             </geometry>
-        </visual>
-<!--        <xacro:if value="${model == 'rubber'}">-->
-           <cylinder length="${wheel_width}" radius="${wheel_radius}"/>
-<!--        </xacro:if>-->
-<!--       <xacro:if value="${model == 'mecanum'}">-->
-<!--          <mesh filename="package://campero_description/meshes/campero_meacanum_a.stl" />-->
-<!--       </xacro:if>-->
+         </visual>
+         <!--        <xacro:if value="${model == 'rubber'}">-->
+         <cylinder length="${wheel_width}" radius="${wheel_radius}" />
+         <!--        </xacro:if>-->
+         <!--       <xacro:if value="${model == 'mecanum'}">-->
+         <!--          <mesh filename="package://campero_description/meshes/campero_meacanum_a.stl" />-->
+         <!--       </xacro:if>-->
       </xacro:chassis>
-      <xacro:if value="${mode == 'simulation' or mode == 'live'}">
-         <xacro:base_control mode="${mode}"/>
-      </xacro:if>
    </xacro:macro>
 </robot>

File: campero_description/urdf/campero_mecanum.urdf.xacro (robot description, xacro)
@@ -3,15 +3,16 @@
   <xacro:arg name="prefix" default="campero_" />
   <xacro:arg name="mode" default="simulation" />
-  <xacro:arg name="controller_conf_yaml_file" default="" />
+  <xacro:arg name="base_name" default="base" />
+  <xacro:arg name="controller_manager_config_yaml_file" default="" />
+  <xacro:arg name="ros2_control_config_urdf_file" default="" />
   <xacro:arg name="ros_prefix" default="/campero/" />
   <xacro:include filename="$(find campero_description)/urdf/campero.xacro" />
   <xacro:campero model="mecanum" mode="$(arg mode)" prefix="$(arg prefix)" />
   <gazebo>
-    <plugin filename="libgazebo_ros2_control.so" name="gazebo_ros2_control">
-      <hardware>$(arg prefix)base</hardware>
-      <robot_param_node>$(arg ros_prefix)robot_state_publisher</robot_param_node>
-      <parameters>$(arg controller_conf_yaml_file)</parameters>
+    <plugin filename="libromea_gazebo_ros2_control.so" name="gazebo_ros2_control">
+      <ros2_control_config_file>$(arg ros2_control_config_urdf_file)</ros2_control_config_file>
+      <controller_manager_config_file>$(arg controller_manager_config_yaml_file)</controller_manager_config_file>
       <ros>
-        <namespace>$(arg ros_prefix)base</namespace>
+        <namespace>$(arg ros_prefix)$(arg base_name)</namespace>
       </ros>
     </plugin>

File: campero_description/urdf/campero_rubber.urdf.xacro (robot description, xacro)
@@ -3,15 +3,16 @@
   <xacro:arg name="prefix" default="campero_" />
   <xacro:arg name="mode" default="simulation" />
-  <xacro:arg name="controller_conf_yaml_file" default="" />
+  <xacro:arg name="base_name" default="base" />
+  <xacro:arg name="controller_manager_config_yaml_file" default="" />
+  <xacro:arg name="ros2_control_config_urdf_file" default="" />
   <xacro:arg name="ros_prefix" default="/campero/" />
   <xacro:include filename="$(find campero_description)/urdf/campero.xacro" />
   <xacro:campero model="rubber" mode="$(arg mode)" prefix="$(arg prefix)" />
   <gazebo>
-    <plugin filename="libgazebo_ros2_control.so" name="gazebo_ros2_control">
-      <hardware>$(arg prefix)base</hardware>
-      <robot_param_node>$(arg ros_prefix)robot_state_publisher</robot_param_node>
-      <parameters>$(arg controller_conf_yaml_file)</parameters>
+    <plugin filename="libromea_gazebo_ros2_control.so" name="gazebo_ros2_control">
+      <ros2_control_config_file>$(arg ros2_control_config_urdf_file)</ros2_control_config_file>
+      <controller_manager_config_file>$(arg controller_manager_config_yaml_file)</controller_manager_config_file>
       <ros>
-        <namespace>$(arg ros_prefix)base</namespace>
+        <namespace>$(arg ros_prefix)$(arg base_name)</namespace>
       </ros>
     </plugin>

Commit message: description: update xacro
Signed-off-by: Jean Laneurit <jean.laneurit@inrae.fr>

File: campero_description/urdf/campero.xacro (robot description, xacro)
@@ -6,8 +6,10 @@
       <xacro:property name="props" value="${load_yaml(conf)}" />
       <!-- Link names -->
-      <xacro:property name="base_link" value="${props['links']['base_link_name']}" />
+      <xacro:property name="base_link"
+         value="${props['links']['base_link_name']}" />
       <xacro:property name="base_footprint_link"
          value="${props['links']['base_footprint_link_name']}" />
-      <xacro:property name="inertial_link" value="${props['links']['inertial_link_name']}" />
+      <xacro:property name="inertial_link"
+         value="${props['links']['inertial_link_name']}" />
       <xacro:property name="front_left_wheel_spinning_link"
          value="${props['links']['front_left_wheel_spinning_link_name']}" />
@@ -32,10 +34,16 @@
          value="${props['joints']['rear_right_wheel_spinning_joint_name']}" />
       <!-- Base Properties -->
-      <xacro:property name="aabb_length" value="${props['geometry']['aabb']['length']}" />
-      <xacro:property name="aabb_width" value="${props['geometry']['aabb']['width']}" />
-      <xacro:property name="aabb_height" value="${props['geometry']['aabb']['height']}" />
-      <xacro:property name="aabb_center_x" value="${props['geometry']['aabb']['center'][0]}" />
-      <xacro:property name="aabb_center_y" value="${props['geometry']['aabb']['center'][1]}" />
-      <xacro:property name="aabb_center_z" value="${props['geometry']['aabb']['center'][2]}" />
+      <xacro:property name="aabb_length"
+         value="${props['geometry']['aabb']['length']}" />
+      <xacro:property name="aabb_width"
+         value="${props['geometry']['aabb']['width']}" />
+      <xacro:property name="aabb_height"
+         value="${props['geometry']['aabb']['height']}" />
+      <xacro:property name="aabb_center_x"
+         value="${props['geometry']['aabb']['center'][0]}" />
+      <xacro:property name="aabb_center_y"
+         value="${props['geometry']['aabb']['center'][1]}" />
+      <xacro:property name="aabb_center_z"
+         value="${props['geometry']['aabb']['center'][2]}" />
       <xacro:property name="wheelbase"
          value="${props['geometry']['axles_distance']}" />
@@ -44,14 +52,20 @@
       <xacro:property name="rear_track"
          value="${props['geometry']['rear_axle']['wheels_distance']}" />
-      <xacro:property name="track"
-         value="${front_track}" />
-      <xacro:property name="ground_clearance" value="${chassis_props['ground_clearance']}" />
-      <xacro:property name="mass_body" value="${props['inertia']['mass']}" />
-      <xacro:property name="mass_base" value="${props['inertia']['mass']}" />
-      <xacro:property name="mass_center_x" value="${props['inertia']['center'][0]}" />
-      <xacro:property name="mass_center_y" value="${props['inertia']['center'][1]}" />
-      <xacro:property name="mass_center_z" value="${props['inertia']['center'][2]}" />
-      <xacro:property name="ground_clearance" value="${props['geometry']['ground_clearance']}" />
-      <xacro:property name="body_reference_x" value="${props['control_point'][0]}" />
+      <!-- <xacro:property name="track"
+         value="${front_track}" /> -->
+      <xacro:property name="mass_body"
+         value="${props['inertia']['mass']}" />
+      <xacro:property name="mass_base"
+         value="${props['inertia']['mass']}" />
+      <xacro:property name="mass_center_x"
+         value="${props['inertia']['center'][0]}" />
+      <xacro:property name="mass_center_y"
+         value="${props['inertia']['center'][1]}" />
+      <xacro:property name="mass_center_z"
+         value="${props['inertia']['center'][2]}" />
+      <xacro:property name="ground_clearance"
+         value="${props['geometry']['ground_clearance']}" />
+      <xacro:property name="body_reference_x"
+         value="${props['control_point'][0]}" />
       <!-- Wheel Properties -->
       <xacro:property name="front_hub_carrier_offset"
@@ -67,6 +81,4 @@
       <xacro:property name="rear_wheel_width"
          value="${props['geometry']['rear_axle']['wheels']['width']}" />
-      <xacro:property name="wheel_radius" value="${front_wheel_radius}" />
-      <xacro:property name="wheel_width" value="${front_wheel_width}" />
       <xacro:property name="maximal_wheel_speed"
          value="${props['wheels_speed_control']['command']['maximal_speed']}" />
@@ -84,8 +96,9 @@
          </visual>
          <!--        <xacro:if value="${model == 'rubber'}">-->
-         <cylinder length="${wheel_width}" radius="${wheel_radius}" />
+         <cylinder length="${front_wheel_width}" radius="${front_wheel_radius}" />
+         <cylinder length="${rear_wheel_width}" radius="${rear_wheel_radius}" />
          <!--        </xacro:if>-->
-         <!--       <xacro:if value="${model == 'mecanum'}">-->
-         <!--          <mesh filename="package://campero_description/meshes/campero_meacanum_a.stl" />-->
+            <!--       <xacro:if value="${model == 'mecanum'}">-->
+            <!--          <mesh filename="package://campero_description/meshes/campero_meacanum_a.stl" />-->
          <!--       </xacro:if>-->
       </xacro:chassis>
