Commit message: description:  add missing properties into ros2_control xacro file
Signed-off-by: jean.laneurit <jean.laneurit@inrae.fr>

File: campero_description/ros2_control/campero.ros2_control.xacro (robot description, xacro)
@@ -20,4 +20,6 @@
     <xacro:property name="rear_wheel_radius"
       value="${props['geometry']['rear_axle']['wheels']['radius']}" />
+    <xacro:property name="maximal_wheel_speed"
+      value="${props['wheels_speed_control']['command']['maximal_speed']}" />
     <!-- simulation plugins -->
     <xacro:if value="${model == 'rubber'}">

Commit message: description: change way to add visuals into xacro file
Signed-off-by: jean.laneurit <jean.laneurit@inrae.fr>

File: campero_description/ros2_control/campero.ros2_control.xacro (robot description, xacro)
@@ -16,4 +16,10 @@
       value="${props['joints']['rear_right_wheel_spinning_joint_name']}" />
     <!-- Geometry -->
+    <xacro:property name="wheelbase"
+      value="${props['geometry']['axles_distance']}" />
+    <xacro:property name="front_track"
+      value="${props['geometry']['front_axle']['wheels_distance']}" />
+    <xacro:property name="rear_track"
+      value="${props['geometry']['rear_axle']['wheels_distance']}" />
     <xacro:property name="front_wheel_radius"
       value="${props['geometry']['front_axle']['wheels']['radius']}" />

File: campero_description/urdf/campero.xacro (robot description, xacro)
@@ -2,4 +2,6 @@
 <robot name="campero" xmlns:xacro="http://www.ros.org/wiki/xacro">
    <xacro:include filename="$(find romea_mobile_base_description)/urdf/base4WD.chassis.xacro" />
+   <xacro:include filename="$(find campero_description)/urdf/visual/chassis.xacro" />
+   <xacro:include filename="$(find campero_description)/urdf/visual/wheels.xacro" />
    <xacro:macro name="campero" params="model mode prefix">
       <xacro:property name="conf" value="$(find campero_description)/config/campero_${model}.yaml" />
@@ -88,18 +90,9 @@
       <xacro:property name="chassis_height" value="${min(front_wheel_radius,rear_wheel_radius)}" />
       <xacro:chassis>
-         <visual>
-            <!--            <origin xyz="${aabb_center_x-body_reference_x} ${aabb_center_y}
-            ${aabb_center_z-chassis_height}" rpy="0 0 0" />-->
-            <geometry>
-               <mesh filename="package://campero_description/meshes/chassis.stl" />
-            </geometry>
-         </visual>
-         <!--        <xacro:if value="${model == 'rubber'}">-->
-         <cylinder length="${front_wheel_width}" radius="${front_wheel_radius}" />
-         <cylinder length="${rear_wheel_width}" radius="${rear_wheel_radius}" />
-         <!--        </xacro:if>-->
-            <!--       <xacro:if value="${model == 'mecanum'}">-->
-            <!--          <mesh filename="package://campero_description/meshes/campero_meacanum_a.stl" />-->
-         <!--       </xacro:if>-->
+         <xacro:chassis_visual />
+         <xacro:front_left_wheel_visual />
+         <xacro:front_right_wheel_visual />
+         <xacro:rear_left_wheel_visual />
+         <xacro:rear_right_wheel_visual />
       </xacro:chassis>
    </xacro:macro>

Commit message: Signed-off-by: Jean Laneurit <jean.laneurit@inrae.fr> merge with bridge

File: campero_description/ros2_control/campero.ros2_control.xacro (robot description, xacro)
@@ -37,5 +37,5 @@
     <xacro:if value="${model == 'mecanum'}">
       <xacro:property name="simulation_hardware_plugin"
-        value="romea_mobile_base_gazebo/GazeboSystemInterface4WMD" />
+        value="romea_mobile_base_gazebo/GazeboSystemInterface4WD" />
       <xacro:property name="live_hardware_plugin"
         value="campero_hardware/CamperoHardware4WMD" />

File: campero_description/urdf/campero_mecanum.urdf.xacro (robot description, xacro)
@@ -5,16 +5,12 @@
   <xacro:arg name="base_name" default="base" />
   <xacro:arg name="controller_manager_config_yaml_file" default="" />
-  <xacro:arg name="ros2_control_config_urdf_file" default="" />
   <xacro:arg name="ros_prefix" default="/campero/" />
   <xacro:include filename="$(find campero_description)/urdf/campero.xacro" />
   <xacro:campero model="mecanum" mode="$(arg mode)" prefix="$(arg prefix)" />
-  <gazebo>
-    <plugin filename="libromea_gazebo_ros2_control.so" name="gazebo_ros2_control">
-      <ros2_control_config_file>$(arg ros2_control_config_urdf_file)</ros2_control_config_file>
-      <controller_manager_config_file>$(arg controller_manager_config_yaml_file)</controller_manager_config_file>
-      <ros>
-        <namespace>$(arg ros_prefix)$(arg base_name)</namespace>
-      </ros>
-    </plugin>
-  </gazebo>
+  <xacro:include filename="$(find campero_description)/urdf/campero.simulation.xacro" />
+  <xacro:campero_simulation
+    mode="$(arg mode)"
+    base_name="$(arg base_name)"
+    ros_prefix="$(arg ros_prefix)"
+    controller_manager_config_yaml_file="$(arg controller_manager_config_yaml_file)" />
 </robot>

File: campero_description/urdf/campero_rubber.urdf.xacro (robot description, xacro)
@@ -5,16 +5,12 @@
   <xacro:arg name="base_name" default="base" />
   <xacro:arg name="controller_manager_config_yaml_file" default="" />
-  <xacro:arg name="ros2_control_config_urdf_file" default="" />
   <xacro:arg name="ros_prefix" default="/campero/" />
   <xacro:include filename="$(find campero_description)/urdf/campero.xacro" />
   <xacro:campero model="rubber" mode="$(arg mode)" prefix="$(arg prefix)" />
-  <gazebo>
-    <plugin filename="libromea_gazebo_ros2_control.so" name="gazebo_ros2_control">
-      <ros2_control_config_file>$(arg ros2_control_config_urdf_file)</ros2_control_config_file>
-      <controller_manager_config_file>$(arg controller_manager_config_yaml_file)</controller_manager_config_file>
-      <ros>
-        <namespace>$(arg ros_prefix)$(arg base_name)</namespace>
-      </ros>
-    </plugin>
-  </gazebo>
+  <xacro:include filename="$(find campero_description)/urdf/campero.simulation.xacro" />
+  <xacro:campero_simulation
+    mode="$(arg mode)"
+    base_name="$(arg base_name)"
+    ros_prefix="$(arg ros_prefix)"
+    controller_manager_config_yaml_file="$(arg controller_manager_config_yaml_file)" />
 </robot>

File: campero_description/urdf/visual/chassis.xacro (robot description, xacro)
@@ -6,5 +6,6 @@
             ${aabb_center_z-chassis_height}" rpy="0 0 0" />-->
             <geometry>
-                <mesh filename="package://campero_description/meshes/chassis.stl" />
+                <!-- <mesh filename="package://campero_description/meshes/chassis.stl" /> -->
+                <mesh filename="file://$(find campero_description)/meshes/chassis.stl" />
             </geometry>
         </visual>
